File: KiCAD/ATX_PSU_525W_ENERMAX/MainsOVPOVPsch.sch (KiCad schematic (older format))
At the start: 12 parts

Commit message: moved all sub schematics to base schematic sheet due to minor complexity
Parts:
- added Q? (x3): Q_NMOS_GDS, symbol Device:Q_NMOS_GDS
- gave numbers to parts that had none: 8
Changed lines of the file:
@@
 +3.3V_IN
 $Comp
-L power:+12V #PWR?
+L power:+12V #PWR0109
 U 1 1 5E06FB81
 P 2000 1450
-F 0 "#PWR?" H 2000 1300 50  0001 C CNN
+F 0 "#PWR0109" H 2000 1300 50  0001 C CNN
 F 1 "+12V" H 2015 1623 50  0000 C CNN
 F 2 "" H 2000 1450 50  0001 C CNN
@@
 $EndComp
 $Comp
-L power:+5V #PWR?
+L power:+5V #PWR0110
 U 1 1 5E0724C2
 P 2000 2800
-F 0 "#PWR?" H 2000 2650 50  0001 C CNN
+F 0 "#PWR0110" H 2000 2650 50  0001 C CNN
 F 1 "+5V" H 2015 2973 50  0000 C CNN
 F 2 "" H 2000 2800 50  0001 C CNN
@@
 $EndComp
 $Comp
-L power:+3.3V #PWR?
+L power:+3.3V #PWR0111
 U 1 1 5E072B74
 P 2000 4250
-F 0 "#PWR?" H 2000 4100 50  0001 C CNN
+F 0 "#PWR0111" H 2000 4100 50  0001 C CNN
 F 1 "+3.3V" H 2015 4423 50  0000 C CNN
 F 2 "" H 2000 4250 50  0001 C CNN
@@
 $EndComp
 $Comp
-L Device:D_Zener_ALT DZ?
+L Device:D_Zener_ALT DZ4
 U 1 1 5E07453E
 P 3700 1700
-F 0 "DZ?" V 3654 1779 50  0000 L CNN
+F 0 "DZ4" V 3654 1779 50  0000 L CNN
 F 1 "D_Zener_ALT" V 3745 1779 50  0000 L CNN
 F 2 "" H 3700 1700 50  0001 C CNN
@@
 $EndComp
 $Comp
-L Device:D_Zener_ALT DZ?
+L Device:D_Zener_ALT DZ5
 U 1 1 5E0750AD
 P 3700 3100
-F 0 "DZ?" V 3654 3179 50  0000 L CNN
+F 0 "DZ5" V 3654 3179 50  0000 L CNN
 F 1 "D_Zener_ALT" V 3745 3179 50  0000 L CNN
 F 2 "" H 3700 3100 50  0001 C CNN
@@
 $EndComp
 $Comp
-L Device:D_Zener_ALT DZ?
+L Device:D_Zener_ALT DZ6
 U 1 1 5E0754FF
 P 3700 4500
-F 0 "DZ?" V 3654 4579 50  0000 L CNN
+F 0 "DZ6" V 3654 4579 50  0000 L CNN
 F 1 "D_Zener_ALT" V 3745 4579 50  0000 L CNN
 F 2 "" H 3700 4500 50  0001 C CNN
@@
 $EndComp
 $Comp
-L power:GNDREF #PWR?
+L power:GNDREF #PWR0112
 U 1 1 5E07598F
 P 3700 2250
-F 0 "#PWR?" H 3700 2000 50  0001 C CNN
+F 0 "#PWR0112" H 3700 2000 50  0001 C CNN
 F 1 "GNDREF" H 3705 2077 50  0000 C CNN
 F 2 "" H 3700 2250 50  0001 C CNN
@@
 $EndComp
 $Comp
-L power:GNDREF #PWR?
+L power:GNDREF #PWR0113
 U 1 1 5E075D9B
 P 3700 3650
-F 0 "#PWR?" H 3700 3400 50  0001 C CNN
+F 0 "#PWR0113" H 3700 3400 50  0001 C CNN
 F 1 "GNDREF" H 3705 3477 50  0000 C CNN
 F 2 "" H 3700 3650 50  0001 C CNN
@@
 $EndComp
 $Comp
-L power:GNDREF #PWR?
+L power:GNDREF #PWR0114
 U 1 1 5E0761B3
 P 3700 5050
-F 0 "#PWR?" H 3700 4800 50  0001 C CNN
+F 0 "#PWR0114" H 3700 4800 50  0001 C CNN
 F 1 "GNDREF" H 3705 4877 50  0000 C CNN
 F 2 "" H 3700 5050 50  0001 C CNN
@@
 AR Path="/5E0B64FB" Ref="D?"  Part="1"
 AR Path="/5E13FF9B/5E0B64FB" Ref="D?"  Part="1"
-AR Path="/5E06D8A7/5E0B64FB" Ref="D?"  Part="1"
-F 0 "D?" H 2700 2700 50  0000 R CNN
+AR Path="/5E06D8A7/5E0B64FB" Ref="D5"  Part="1"
+F 0 "D5" H 2700 2700 50  0000 R CNN
 F 1 "20A" H 2700 2900 50  0000 R CNN
 F 2 "Diode_SMD_STMicroelectronics:DPAK228P972X240-3N" H 2650 2800 50  0001 C CNN
@@
 AR Path="/5E0B68E4" Ref="D?"  Part="1"
 AR Path="/5E13FF9B/5E0B68E4" Ref="D?"  Part="1"
-AR Path="/5E06D8A7/5E0B68E4" Ref="D?"  Part="1"
-F 0 "D?" H 2700 4150 50  0000 R CNN
+AR Path="/5E06D8A7/5E0B68E4" Ref="D6"  Part="1"
+F 0 "D6" H 2700 4150 50  0000 R CNN
 F 1 "20A" H 2700 4350 50  0000 R CNN
 F 2 "Diode_SMD_STMicroelectronics:DPAK228P972X240-3N" H 2650 4250 50  0001 C CNN
@@
 P 3700 2100
 AR Path="/5E13FF9B/5E0BF0E0" Ref="R?"  Part="1"
-AR Path="/5E06D8A7/5E0BF0E0" Ref="R?"  Part="1"
-F 0 "R?" H 3770 2146 50  0000 L CNN
+AR Path="/5E06D8A7/5E0BF0E0" Ref="R4"  Part="1"
+F 0 "R4" H 3770 2146 50  0000 L CNN
 F 1 "1M" V 3700 2050 50  0000 L CNN
 F 2 "Resistor_THT:R_Axial_DIN0516_L15.5mm_D5.0mm_P20.32mm_Horizontal" V 3630 2100 50  0001 C CNN
@@
 P 3700 3500
 AR Path="/5E13FF9B/5E0BF537" Ref="R?"  Part="1"
-AR Path="/5E06D8A7/5E0BF537" Ref="R?"  Part="1"
-F 0 "R?" H 3770 3546 50  0000 L CNN
+AR Path="/5E06D8A7/5E0BF537" Ref="R5"  Part="1"
+F 0 "R5" H 3770 3546 50  0000 L CNN
 F 1 "1M" V 3700 3450 50  0000 L CNN
 F 2 "Resistor_THT:R_Axial_DIN0516_L15.5mm_D5.0mm_P20.32mm_Horizontal" V 3630 3500 50  0001 C CNN
@@
 P 3700 4900
 AR Path="/5E13FF9B/5E0BFC05" Ref="R?"  Part="1"
-AR Path="/5E06D8A7/5E0BFC05" Ref="R?"  Part="1"
-F 0 "R?" H 3770 4946 50  0000 L CNN
+AR Path="/5E06D8A7/5E0BFC05" Ref="R6"  Part="1"
+F 0 "R6" H 3770 4946 50  0000 L CNN
 F 1 "1M" V 3700 4850 50  0000 L CNN
 F 2 "Resistor_THT:R_Axial_DIN0516_L15.5mm_D5.0mm_P20.32mm_Horizontal" V 3630 4900 50  0001 C CNN
@@
 	1    0    0    -1
 $EndComp
+$Comp
+L Device:Q_NMOS_GDS Q?
+U 1 1 6160A41E
+P 4600 1950
+F 0 "Q?" H 4804 1996 50  0000 L CNN
+F 1 "Q_NMOS_GDS" H 4804 1905 50  0000 L CNN
+F 2 "" H 4800 2050 50  0001 C CNN
+F 3 "~" H 4600 1950 50  0001 C CNN
+	1    4600 1950
+	1    0    0    -1
+$EndComp
+$Comp
+L Device:Q_NMOS_GDS Q?
+U 1 1 6160BD61
+P 4650 3400
+F 0 "Q?" H 4854 3446 50  0000 L CNN
+F 1 "Q_NMOS_GDS" H 4854 3355 50  0000 L CNN
+F 2 "" H 4850 3500 50  0001 C CNN
+F 3 "~" H 4650 3400 50  0001 C CNN
+	1    4650 3400
+	1    0    0    -1
+$EndComp
+$Comp
+L Device:Q_NMOS_GDS Q?
+U 1 1 6160C62E
+P 4600 4700
+F 0 "Q?" H 4804 4746 50  0000 L CNN
+F 1 "Q_NMOS_GDS" H 4804 4655 50  0000 L CNN
+F 2 "" H 4800 4800 50  0001 C CNN
+F 3 "~" H 4600 4700 50  0001 C CNN
+	1    4600 4700
+	1    0    0    -1
+$EndComp
