File: KiCAD/ATX_PSU_525W_ENERMAX/ATX_PSU_525W_ENERMAX.sch (KiCad schematic (older format))
At the start: 87 parts, among them J1 Fan1, J10 EPS12V 8 Pin, J11 Current Sens, J12 Molex: 0039281243, J13 Molex: 0039281243, J14 Molex: 0039281243, J15 Potti, J16 Potti, J17 LED Yellow, J18 LED Yellow, J19 Volt Sens, J2 Power On Switch, J20 12V Out, J21 Volt Sens, J22 12V Out, J23 Molex: 0039281243, J24 Current Sens, J25 Current Sens, J26 Molex: 0039281243, J27 Molex: 0039281243, J28 Fan1, J29 Fan1, J3 Standby LED, J30 Potti, J31 Potti, J32 LED Red, J33 LED Orange, J34 Volt Sens, J35 5V Out, J36 Volt Sens, J37 3.3V Out, J38 Screw_Terminal_01x06, J39 Screw_Terminal_01x06, J4 EPS12V 4Pin, J40 Current Sens, J41 Current Sens, J42 Screw_Terminal_01x06, J43 Screw_Terminal_01x06, J44 Screw_Terminal_01x12, J5 Potti, J6 LED Yellow, J7 Volt Sens, J8 12V Out, J9 Main ATX 24Pin, Q1 Q_NMOS_DGS, Q2 Q_NMOS_DGS, Q3 Q_NMOS_DGS, Q4 Q_NMOS_DGS, Q5 Q_NMOS_DGS, U1 ACS712xLCTR-20A, U2 ACS712xLCTR-20A, U3 ACS712xLCTR-20A, U4 ACS712xLCTR-20A, U5 ACS712xLCTR-20A

Commit message: performed rule check
Connections:
- net +5V: no longer DZ4.1 (K), F4.2, J28.1 (Pin_1), R10.2, R9.1, U4.1 (IP+), U4.2 (IP+)
- removed net +12V: DZ1.1 (K), DZ2.1 (K), DZ3.1 (K), F1.2, F2.2, F3.2, J1.1 (Pin_1), R1.1, R2.1, R3.2, R5.1, R6.2, R7.1, R8.2, U1.1 (IP+), U1.2 (IP+), U2.1 (IP+), U2.2 (IP+), U3.1 (IP+), U3.2 (IP+)
- net +3V3: no longer names the net of DZ5.1 (K), F5.2, J29.1 (Pin_1), R11.1, R12.2, U5.1 (IP+), U5.2 (IP+)
- new net: DZ1.1 (K), F1.2, J1.1 (Pin_1), R1.1, R2.1, R3.2, U1.1 (IP+), U1.2 (IP+)
- new net: DZ2.1 (K), F2.2, R5.1, R6.2, U2.1 (IP+), U2.2 (IP+)
- new net: DZ3.1 (K), F3.2, R7.1, R8.2, U3.1 (IP+), U3.2 (IP+)
- new net: DZ4.1 (K), F4.2, J28.1 (Pin_1), R10.2, R9.1, U4.1 (IP+), U4.2 (IP+)
- no-connect marks 4 -> 6
Other:
- note added: "These pins will not \nbe used in the \npower supply"
- moved on the sheet: J10, J12, J13, J14, J23, J26, J27, J38, J39, J4, J42, J43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

Commit message: Assigned pcb footprints
Parts:
- C1, C10, C2, C3, C4, C5, C6, C7, C8, C9: footprint (none) -> Capacitor_SMD:C_0603_1608Metric_Pad1.05x0.95mm_HandSolder
- DZ1, DZ2, DZ3, DZ4, DZ5: footprint (none) -> Diode_SMD:D_SMC_Handsoldering
- J12, J14, J27: footprint Connector_Molex:Molex_Mini-Fit_Jr_5566-08A2_2x04_P4.20mm_Vertical -> Connector_Molex:Molex_Mini-Fit_Jr_5566-08A_2x04_P4.20mm_Vertical
- J38, J39, J42, J43: footprint (none) -> TerminalBlock_RND:TerminalBlock_RND_205-00005_1x06_P5.00mm_Horizontal
- J4: footprint (none) -> Connector_Molex:Molex_Mini-Fit_Jr_5566-04A_2x02_P4.20mm_Vertical
- J44: footprint (none) -> TerminalBlock_RND:TerminalBlock_RND_205-00011_1x12_P5.00mm_Horizontal
- R1, R11, R4, R5, R9: footprint Resistor_THT:R_Axial_Power_L20.0mm_W6.4mm_P25.40mm -> Resistor_THT:R_Axial_DIN0516_L15.5mm_D5.0mm_P20.32mm_Horizontal
Changed lines of the file:
@@
 F 0 "J38" V 1400 5800 50  0000 R CNN
 F 1 "Screw_Terminal_01x06" V 1300 6150 50  0000 R CNN
-F 2 "" H 1200 5800 50  0001 C CNN
+F 2 "TerminalBlock_RND:TerminalBlock_RND_205-00005_1x06_P5.00mm_Horizontal" H 1200 5800 50  0001 C CNN
 F 3 "~" H 1200 5800 50  0001 C CNN
 	1    1200 5800
@@
 F 0 "J39" V 2450 5800 50  0000 R CNN
 F 1 "Screw_Terminal_01x06" V 2350 6150 50  0000 R CNN
-F 2 "" H 2250 5800 50  0001 C CNN
+F 2 "TerminalBlock_RND:TerminalBlock_RND_205-00005_1x06_P5.00mm_Horizontal" H 2250 5800 50  0001 C CNN
 F 3 "~" H 2250 5800 50  0001 C CNN
 	1    2250 5800
@@
 F 0 "J42" V 1400 6550 50  0000 R CNN
 F 1 "Screw_Terminal_01x06" V 1300 6900 50  0000 R CNN
-F 2 "" H 1200 6550 50  0001 C CNN
+F 2 "TerminalBlock_RND:TerminalBlock_RND_205-00005_1x06_P5.00mm_Horizontal" H 1200 6550 50  0001 C CNN
 F 3 "~" H 1200 6550 50  0001 C CNN
 	1    1200 6550
@@
 F 0 "J43" V 2450 6550 50  0000 R CNN
 F 1 "Screw_Terminal_01x06" V 2350 6900 50  0000 R CNN
-F 2 "" H 2250 6550 50  0001 C CNN
+F 2 "TerminalBlock_RND:TerminalBlock_RND_205-00005_1x06_P5.00mm_Horizontal" H 2250 6550 50  0001 C CNN
 F 3 "~" H 2250 6550 50  0001 C CNN
 	1    2250 6550
@@
 F 0 "J44" V 1967 7246 50  0000 C CNN
 F 1 "Screw_Terminal_01x12" V 1876 7246 50  0000 C CNN
-F 2 "" H 1750 7300 50  0001 C CNN
+F 2 "TerminalBlock_RND:TerminalBlock_RND_205-00011_1x12_P5.00mm_Horizontal" H 1750 7300 50  0001 C CNN
 F 3 "~" H 1750 7300 50  0001 C CNN
 	1    1750 7300
@@
 F 0 "J4" H 3000 625 50  0000 C CNN
 F 1 "EPS12V 4Pin" H 3000 716 50  0000 C CNN
-F 2 "" H 2950 950 50  0001 C CNN
+F 2 "Connector_Molex:Molex_Mini-Fit_Jr_5566-04A_2x02_P4.20mm_Vertical" H 2950 950 50  0001 C CNN
 F 3 "~" H 2950 950 50  0001 C CNN
 	1    2950 950
@@
 F 0 "J27" H 1200 4750 50  0000 C CNN
 F 1 "Molex: 0039281243" V 1200 4900 39  0001 C CNN
-F 2 "Connector_Molex:Molex_Mini-Fit_Jr_5566-08A2_2x04_P4.20mm_Vertical" H 1150 4950 50  0001 C CNN
+F 2 "Connector_Molex:Molex_Mini-Fit_Jr_5566-08A_2x04_P4.20mm_Vertical" H 1150 4950 50  0001 C CNN
 F 3 "https://www.molex.com/pdm_docs/sd/039281243_sd.pdf" H 1150 4950 50  0001 C CNN
 F 4 "WM3811-ND " H 1200 5250 50  0001 C CNN "Digi-Key"
@@
 F 0 "C6" H 9450 3800 50  0000 R CNN
 F 1 "0.1uF" H 9500 3900 50  0000 R CNN
-F 2 "" H 9588 3650 50  0001 C CNN
+F 2 "Capacitor_SMD:C_0603_1608Metric_Pad1.05x0.95mm_HandSolder" H 9588 3650 50  0001 C CNN
 F 3 "~" H 9550 3800 50  0001 C CNN
 	1    9550 3800
@@
 F 0 "C4" V 10050 3750 50  0000 C CNN
 F 1 "1nF" V 10350 3750 50  0000 C CNN
-F 2 "" H 10238 3600 50  0001 C CNN
+F 2 "Capacitor_SMD:C_0603_1608Metric_Pad1.05x0.95mm_HandSolder" H 10238 3600 50  0001 C CNN
 F 3 "~" H 10200 3750 50  0001 C CNN
 	1    10200 3750
@@
 F 0 "DZ3" V 8500 3050 50  0000 L CNN
 F 1 "D_Zener_ALT" V 8545 3079 50  0001 L CNN
-F 2 "" H 8500 3000 50  0001 C CNN
+F 2 "Diode_SMD:D_SMC_Handsoldering" H 8500 3000 50  0001 C CNN
 F 3 "~" H 8500 3000 50  0001 C CNN
 	1    8500 3000
@@
 F 0 "C10" H 9450 5800 50  0000 R CNN
 F 1 "0.1uF" H 9500 5900 50  0000 R CNN
-F 2 "" H 9588 5650 50  0001 C CNN
+F 2 "Capacitor_SMD:C_0603_1608Metric_Pad1.05x0.95mm_HandSolder" H 9588 5650 50  0001 C CNN
 F 3 "~" H 9550 5800 50  0001 C CNN
 	1    9550 5800
@@
 F 0 "C8" V 10050 5750 50  0000 C CNN
 F 1 "1nF" V 10350 5750 50  0000 C CNN
-F 2 "" H 10238 5600 50  0001 C CNN
+F 2 "Capacitor_SMD:C_0603_1608Metric_Pad1.05x0.95mm_HandSolder" H 10238 5600 50  0001 C CNN
 F 3 "~" H 10200 5750 50  0001 C CNN
 	1    10200 5750
@@
 F 0 "R11" H 8000 5000 50  0000 L CNN
 F 1 "20" V 7950 4950 50  0000 L CNN
-F 2 "Resistor_THT:R_Axial_Power_L20.0mm_W6.4mm_P25.40mm" V 7880 5000 50  0001 C CNN
+F 2 "Resistor_THT:R_Axial_DIN0516_L15.5mm_D5.0mm_P20.32mm_Horizontal" V 7880 5000 50  0001 C CNN
 F 3 "~" H 7950 5000 50  0001 C CNN
 	1    7950 5000
@@
 F 0 "DZ5" V 8200 5050 50  0000 L CNN
 F 1 "D_Zener_ALT" V 8245 5079 50  0001 L CNN
-F 2 "" H 8200 5000 50  0001 C CNN
+F 2 "Diode_SMD:D_SMC_Handsoldering" H 8200 5000 50  0001 C CNN
 F 3 "~" H 8200 5000 50  0001 C CNN
 	1    8200 5000
@@
 F 0 "R9" H 4050 5000 50  0000 L CNN
 F 1 "300" V 4000 4950 50  0000 L CNN
-F 2 "Resistor_THT:R_Axial_Power_L20.0mm_W6.4mm_P25.40mm" V 3930 5000 50  0001 C CNN
+F 2 "Resistor_THT:R_Axial_DIN0516_L15.5mm_D5.0mm_P20.32mm_Horizontal" V 3930 5000 50  0001 C CNN
 F 3 "~" H 4000 5000 50  0001 C CNN
 	1    4000 5000
@@
 F 0 "DZ4" V 4250 5050 50  0000 L CNN
 F 1 "D_Zener_ALT" V 4295 5079 50  0001 L CNN
-F 2 "" H 4250 5000 50  0001 C CNN
+F 2 "Diode_SMD:D_SMC_Handsoldering" H 4250 5000 50  0001 C CNN
 F 3 "~" H 4250 5000 50  0001 C CNN
 	1    4250 5000
@@
 F 0 "C7" V 6100 5750 50  0000 C CNN
 F 1 "1nF" V 6400 5750 50  0000 C CNN
-F 2 "" H 6288 5600 50  0001 C CNN
+F 2 "Capacitor_SMD:C_0603_1608Metric_Pad1.05x0.95mm_HandSolder" H 6288 5600 50  0001 C CNN
 F 3 "~" H 6250 5750 50  0001 C CNN
 	1    6250 5750
@@
 F 0 "C9" H 5500 5800 50  0000 R CNN
 F 1 "0.1uF" H 5550 5900 50  0000 R CNN
-F 2 "" H 5638 5650 50  0001 C CNN
+F 2 "Capacitor_SMD:C_0603_1608Metric_Pad1.05x0.95mm_HandSolder" H 5638 5650 50  0001 C CNN
 F 3 "~" H 5600 5800 50  0001 C CNN
 	1    5600 5800
@@
 F 0 "R5" H 4350 3000 50  0000 L CNN
 F 1 "680" V 4300 2950 50  0000 L CNN
-F 2 "Resistor_THT:R_Axial_Power_L20.0mm_W6.4mm_P25.40mm" V 4230 3000 50  0001 C CNN
+F 2 "Resistor_THT:R_Axial_DIN0516_L15.5mm_D5.0mm_P20.32mm_Horizontal" V 4230 3000 50  0001 C CNN
 F 3 "~" H 4300 3000 50  0001 C CNN
 	1    4300 3000
@@
 F 0 "DZ2" V 4550 3050 50  0000 L CNN
 F 1 "D_Zener_ALT" V 4595 3079 50  0001 L CNN
-F 2 "" H 4550 3000 50  0001 C CNN
+F 2 "Diode_SMD:D_SMC_Handsoldering" H 4550 3000 50  0001 C CNN
 F 3 "~" H 4550 3000 50  0001 C CNN
 	1    4550 3000
@@
 F 0 "C3" V 6100 3750 50  0000 C CNN
 F 1 "1nF" V 6300 3600 50  0000 C CNN
-F 2 "" H 6288 3600 50  0001 C CNN
+F 2 "Capacitor_SMD:C_0603_1608Metric_Pad1.05x0.95mm_HandSolder" H 6288 3600 50  0001 C CNN
 F 3 "~" H 6250 3750 50  0001 C CNN
 	1    6250 3750
@@
 F 0 "C5" H 5500 3800 50  0000 R CNN
 F 1 "0.1uF" H 5550 3900 50  0000 R CNN
-F 2 "" H 5638 3650 50  0001 C CNN
+F 2 "Capacitor_SMD:C_0603_1608Metric_Pad1.05x0.95mm_HandSolder" H 5638 3650 50  0001 C CNN
 F 3 "~" H 5600 3800 50  0001 C CNN
 	1    5600 3800
@@
 F 0 "R1" H 7700 1000 50  0000 L CNN
 F 1 "680" V 7650 950 50  0000 L CNN
-F 2 "Resistor_THT:R_Axial_Power_L20.0mm_W6.4mm_P25.40mm" V 7580 1000 50  0001 C CNN
+F 2 "Resistor_THT:R_Axial_DIN0516_L15.5mm_D5.0mm_P20.32mm_Horizontal" V 7580 1000 50  0001 C CNN
 F 3 "~" H 7650 1000 50  0001 C CNN
 	1    7650 1000
@@
 F 0 "DZ1" V 8200 1050 50  0000 L CNN
 F 1 "D_Zener_ALT" V 8245 1079 50  0001 L CNN
-F 2 "" H 8200 1000 50  0001 C CNN
+F 2 "Diode_SMD:D_SMC_Handsoldering" H 8200 1000 50  0001 C CNN
 F 3 "~" H 8200 1000 50  0001 C CNN
 	1    8200 1000
@@
 F 0 "C1" V 10050 1750 50  0000 C CNN
 F 1 "1nF" V 10350 1750 50  0000 C CNN
-F 2 "" H 10238 1600 50  0001 C CNN
+F 2 "Capacitor_SMD:C_0603_1608Metric_Pad1.05x0.95mm_HandSolder" H 10238 1600 50  0001 C CNN
 F 3 "~" H 10200 1750 50  0001 C CNN
 	1    10200 1750
@@
 F 0 "R4" H 5650 1350 50  0000 L CNN
 F 1 "680" V 5600 1300 50  0000 L CNN
-F 2 "Resistor_THT:R_Axial_Power_L20.0mm_W6.4mm_P25.40mm" V 5530 1350 50  0001 C CNN
+F 2 "Resistor_THT:R_Axial_DIN0516_L15.5mm_D5.0mm_P20.32mm_Horizontal" V 5530 1350 50  0001 C CNN
 F 3 "~" H 5600 1350 50  0001 C CNN
 	1    5600 1350
@@
 F 0 "C2" H 9450 1800 50  0000 R CNN
 F 1 "0.1uF" H 9500 1900 50  0000 R CNN
-F 2 "" H 9588 1650 50  0001 C CNN
+F 2 "Capacitor_SMD:C_0603_1608Metric_Pad1.05x0.95mm_HandSolder" H 9588 1650 50  0001 C CNN
 F 3 "~" H 9550 1800 50  0001 C CNN
 	1    9550 1800
@@
 F 0 "J14" H 1200 3400 50  0000 C CNN
 F 1 "Molex: 0039281243" V 1200 3550 39  0001 C CNN
-F 2 "Connector_Molex:Molex_Mini-Fit_Jr_5566-08A2_2x04_P4.20mm_Vertical" H 1150 3600 50  0001 C CNN
+F 2 "Connector_Molex:Molex_Mini-Fit_Jr_5566-08A_2x04_P4.20mm_Vertical" H 1150 3600 50  0001 C CNN
 F 3 "https://www.molex.com/pdm_docs/sd/039281243_sd.pdf" H 1150 3600 50  0001 C CNN
 F 4 "WM3811-ND " H 1200 3900 50  0001 C CNN "Digi-Key"
@@
 F 0 "J12" H 1200 2850 50  0000 C CNN
 F 1 "Molex: 0039281243" V 1200 3000 39  0001 C CNN
-F 2 "Connector_Molex:Molex_Mini-Fit_Jr_5566-08A2_2x04_P4.20mm_Vertical" H 1150 3050 50  0001 C CNN
+F 2 "Connector_Molex:Molex_Mini-Fit_Jr_5566-08A_2x04_P4.20mm_Vertical" H 1150 3050 50  0001 C CNN
 F 3 "https://www.molex.com/pdm_docs/sd/039281243_sd.pdf" H 1150 3050 50  0001 C CNN
 F 4 "WM3811-ND " H 1200 2800 50  0001 C CNN "Digi-Key"
