File: KiCAD/ATX_PSU_525W_ENERMAX/ATX_PSDB.sch (KiCad schematic (older format))
At the start: 87 parts, among them J1 Fan1, J10 EPS12V 8 Pin, J11 Current Sens, J12 Molex: 0039281243, J13 Molex: 0039281243, J14 Molex: 0039281243, J15 Potti, J16 Potti, J17 LED Yellow, J18 LED Yellow, J19 Volt Sens, J2 Power On Switch, J20 12V Out, J21 Volt Sens, J22 12V Out, J23 Molex: 0039281243, J24 Current Sens, J25 Current Sens, J26 Molex: 0039281243, J27 Molex: 0039281243, J28 Fan1, J29 Fan1, J3 Standby LED, J30 Potti, J31 Potti, J32 LED Red, J33 LED Orange, J34 Volt Sens, J35 5V Out, J36 Volt Sens, J37 3.3V Out, J38 Screw_Terminal_01x06, J39 Screw_Terminal_01x06, J4 EPS12V 4Pin, J40 Current Sens, J41 Current Sens, J42 Screw_Terminal_01x06, J43 Screw_Terminal_01x06, J44 Screw_Terminal_01x12, J5 Potti, J6 LED Yellow, J7 Volt Sens, J8 12V Out, J9 Main ATX 24Pin, Q1 Q_NMOS_DGS, Q2 Q_NMOS_DGS, Q3 Q_NMOS_DGS, Q4 Q_NMOS_DGS, Q5 Q_NMOS_DGS, U1 ACS712xLCTR-20A, U2 ACS712xLCTR-20A, U3 ACS712xLCTR-20A, U4 ACS712xLCTR-20A, U5 ACS712xLCTR-20A

Commit message: some cleanup
Parts:
- J12, J14, J27: footprint Connector_Molex:Molex_Mini-Fit_Jr_5566-08A_2x04_P4.20mm_Vertical -> Connector_Molex:Molex_Mini-Fit_Jr_5566-06A_2x03_P4.20mm_Vertical
- J23: footprint Connector_Molex:Molex_Mini-Fit_Jr_5566-08A2_2x04_P4.20mm_Vertical -> Connector_Molex:Molex_Mini-Fit_Jr_5566-06A_2x03_P4.20mm_Vertical
Other:
- note added: "Ground Terminal"
- note added: "Secondary +5V and +3.3V Power Input Terminal"
- note removed: "Secondary +5V Power Input Terminal"
Changed lines of the file:
@@
 Sheet 1 1
 Title "ATX Power Supply Distribution Board"
-Date ""
-Rev ""
+Date "2022-03-01"
+Rev "1.0"
 Comp "Ibrahim Tüzenli"
 Comment1 ""
@@
 	2250 7500 2150 7500
 Text Notes 1050 6250 0    50   ~ 0
-Secondary +5V Power Input Terminal
+Secondary +5V and +3.3V Power Input Terminal
 Text Notes 800  7000 0    50   ~ 0
-Secondary +12V2/+12V3 Power Rail Input Terminal
+Ground Terminal
 Wire Wire Line
 	1200 6000 1300 6000
@@
 F 0 "J23" H 1200 4200 50  0000 C CNN
 F 1 "Molex: 0039281243" V 1200 4350 39  0001 C CNN
-F 2 "Connector_Molex:Molex_Mini-Fit_Jr_5566-08A2_2x04_P4.20mm_Vertical" H 1150 4400 50  0001 C CNN
+F 2 "Connector_Molex:Molex_Mini-Fit_Jr_5566-06A_2x03_P4.20mm_Vertical" H 1150 4400 50  0001 C CNN
 F 3 "https://www.molex.com/pdm_docs/sd/039281243_sd.pdf" H 1150 4400 50  0001 C CNN
 F 4 "WM3811-ND " H 1200 4150 50  0001 C CNN "Digi-Key"
@@
 F 0 "J27" H 1200 4750 50  0000 C CNN
 F 1 "Molex: 0039281243" V 1200 4900 39  0001 C CNN
-F 2 "Connector_Molex:Molex_Mini-Fit_Jr_5566-08A_2x04_P4.20mm_Vertical" H 1150 4950 50  0001 C CNN
+F 2 "Connector_Molex:Molex_Mini-Fit_Jr_5566-06A_2x03_P4.20mm_Vertical" H 1150 4950 50  0001 C CNN
 F 3 "https://www.molex.com/pdm_docs/sd/039281243_sd.pdf" H 1150 4950 50  0001 C CNN
 F 4 "WM3811-ND " H 1200 5250 50  0001 C CNN "Digi-Key"
@@
 F 1 "10A" V 7900 2950 50  0000 R CNN
 F 2 "Fuse:Fuseholder_Cylinder-6.3x32mm_Schurter_0031-8002_Horizontal_Open" V 7930 2850 50  0001 C CNN
-F 3 "https://us.schurter.com/en/datasheet/typ_SHF_6.3x32.pdf / https://us.schurter.com/bundles/snceschurter/epim/_ProdPool_/newDS/en/typ_OG__Holder__6.3x32.pdf" H 8000 2850 50  0001 C CNN
+F 3 "https://us.schurter.com/en/datasheet/typ_SHF_6.3x32.pdf" H 8000 2850 50  0001 C CNN
 F 4 "486-3322-ND / 486-3643-ND" H 8000 2850 50  0001 C CNN "DigiKey_Nr"
 F 5 "Schurter Inc" H 8000 2850 50  0001 C CNN "OEM"
@@
 F 1 "10A" V 7600 4950 50  0000 R CNN
 F 2 "Fuse:Fuseholder_Cylinder-6.3x32mm_Schurter_0031-8002_Horizontal_Open" V 7630 4850 50  0001 C CNN
-F 3 "https://us.schurter.com/en/datasheet/typ_SHF_6.3x32.pdf / https://us.schurter.com/bundles/snceschurter/epim/_ProdPool_/newDS/en/typ_OG__Holder__6.3x32.pdf" H 7700 4850 50  0001 C CNN
+F 3 "https://us.schurter.com/en/datasheet/typ_SHF_6.3x32.pdf" H 7700 4850 50  0001 C CNN
 F 4 "486-3322-ND / 486-3643-ND" H 7700 4850 50  0001 C CNN "DigiKey_Nr"
 F 5 "Schurter Inc" H 7700 4850 50  0001 C CNN "OEM"
@@
 F 1 "10A" V 3650 4950 50  0000 R CNN
 F 2 "Fuse:Fuseholder_Cylinder-6.3x32mm_Schurter_0031-8002_Horizontal_Open" V 3680 4850 50  0001 C CNN
-F 3 "https://us.schurter.com/en/datasheet/typ_SHF_6.3x32.pdf / https://us.schurter.com/bundles/snceschurter/epim/_ProdPool_/newDS/en/typ_OG__Holder__6.3x32.pdf" H 3750 4850 50  0001 C CNN
+F 3 "https://us.schurter.com/en/datasheet/typ_SHF_6.3x32.pdf" H 3750 4850 50  0001 C CNN
 F 4 "486-3322-ND / 486-3643-ND" H 3750 4850 50  0001 C CNN "DigiKey_Nr"
 F 5 "Schurter Inc" H 3750 4850 50  0001 C CNN "OEM"
@@
 F 1 "10A" V 3950 2950 50  0000 R CNN
 F 2 "Fuse:Fuseholder_Cylinder-6.3x32mm_Schurter_0031-8002_Horizontal_Open" V 3980 2850 50  0001 C CNN
-F 3 "https://us.schurter.com/en/datasheet/typ_SHF_6.3x32.pdf / https://us.schurter.com/bundles/snceschurter/epim/_ProdPool_/newDS/en/typ_OG__Holder__6.3x32.pdf" H 4050 2850 50  0001 C CNN
+F 3 "https://us.schurter.com/en/datasheet/typ_SHF_6.3x32.pdf" H 4050 2850 50  0001 C CNN
 F 4 "486-3322-ND / 486-3643-ND" H 4050 2850 50  0001 C CNN "DigiKey_Nr"
 F 5 "Schurter Inc" H 4050 2850 50  0001 C CNN "OEM"
@@
 F 1 "10A" V 7350 950 50  0000 R CNN
 F 2 "Fuse:Fuseholder_Cylinder-6.3x32mm_Schurter_0031-8002_Horizontal_Open" V 7380 850 50  0001 C CNN
-F 3 "https://us.schurter.com/en/datasheet/typ_SHF_6.3x32.pdf / https://us.schurter.com/bundles/snceschurter/epim/_ProdPool_/newDS/en/typ_OG__Holder__6.3x32.pdf" H 7450 850 50  0001 C CNN
+F 3 "https://us.schurter.com/en/datasheet/typ_SHF_6.3x32.pdf" H 7450 850 50  0001 C CNN
 F 4 "486-3322-ND / 486-3643-ND" H 7450 850 50  0001 C CNN "DigiKey_Nr"
 F 5 "Schurter Inc" H 7450 850 50  0001 C CNN "OEM"
@@
 F 0 "J14" H 1200 3400 50  0000 C CNN
 F 1 "Molex: 0039281243" V 1200 3550 39  0001 C CNN
-F 2 "Connector_Molex:Molex_Mini-Fit_Jr_5566-08A_2x04_P4.20mm_Vertical" H 1150 3600 50  0001 C CNN
+F 2 "Connector_Molex:Molex_Mini-Fit_Jr_5566-06A_2x03_P4.20mm_Vertical" H 1150 3600 50  0001 C CNN
 F 3 "https://www.molex.com/pdm_docs/sd/039281243_sd.pdf" H 1150 3600 50  0001 C CNN
 F 4 "WM3811-ND " H 1200 3900 50  0001 C CNN "Digi-Key"
@@
 F 0 "J12" H 1200 2850 50  0000 C CNN
 F 1 "Molex: 0039281243" V 1200 3000 39  0001 C CNN
-F 2 "Connector_Molex:Molex_Mini-Fit_Jr_5566-08A_2x04_P4.20mm_Vertical" H 1150 3050 50  0001 C CNN
+F 2 "Connector_Molex:Molex_Mini-Fit_Jr_5566-06A_2x03_P4.20mm_Vertical" H 1150 3050 50  0001 C CNN
 F 3 "https://www.molex.com/pdm_docs/sd/039281243_sd.pdf" H 1150 3050 50  0001 C CNN
 F 4 "WM3811-ND " H 1200 2800 50  0001 C CNN "Digi-Key"

Commit message: changed terminal blocks to wago footprints
Parts:
- J10: footprint Connector_Molex:Molex_Mini-Fit_Jr_5566-12A_2x06_P4.20mm_Vertical -> Connector_Molex:Molex_Mini-Fit_Jr_5566-08A_2x04_P4.20mm_Vertical
- J20, J22, J35, J37, J8: footprint TerminalBlock_Altech:Altech_AK300_1x02_P5.00mm_45-Degree -> TerminalBlock_WAGO:TerminalBlock_WAGO_236-102_1x02_P5.00mm_45Degree
- J38, J39, J42, J43: footprint TerminalBlock_RND:TerminalBlock_RND_205-00005_1x06_P5.00mm_Horizontal -> TerminalBlock_WAGO:TerminalBlock_WAGO_236-108_1x08_P5.00mm_45Degree
- J44: footprint TerminalBlock_RND:TerminalBlock_RND_205-00011_1x12_P5.00mm_Horizontal -> TerminalBlock_WAGO:TerminalBlock_WAGO_236-112_1x12_P5.00mm_45Degree
- R7: footprint Resistor_THT:R_Axial_Power_L20.0mm_W6.4mm_P25.40mm -> Resistor_THT:R_Axial_DIN0516_L15.5mm_D5.0mm_P20.32mm_Horizontal
Changed lines of the file:
@@
 F 0 "J10" H 3000 1200 50  0000 C CNN
 F 1 "EPS12V 8 Pin" H 3000 1300 50  0000 C CNN
-F 2 "Connector_Molex:Molex_Mini-Fit_Jr_5566-12A_2x06_P4.20mm_Vertical" H 2950 1600 50  0001 C CNN
+F 2 "Connector_Molex:Molex_Mini-Fit_Jr_5566-08A_2x04_P4.20mm_Vertical" H 2950 1600 50  0001 C CNN
 F 3 "https://www.molex.com/pdm_docs/sd/039281243_sd.pdf" H 2950 1600 50  0001 C CNN
 F 4 "WM3811-ND " H 3050 1850 50  0001 C CNN "Digi-Key"
@@
 F 0 "J38" V 1400 5800 50  0000 R CNN
 F 1 "Screw_Terminal_01x06" V 1300 6150 50  0000 R CNN
-F 2 "TerminalBlock_RND:TerminalBlock_RND_205-00005_1x06_P5.00mm_Horizontal" H 1200 5800 50  0001 C CNN
+F 2 "TerminalBlock_WAGO:TerminalBlock_WAGO_236-108_1x08_P5.00mm_45Degree" H 1200 5800 50  0001 C CNN
 F 3 "~" H 1200 5800 50  0001 C CNN
 	1    1200 5800
@@
 F 0 "J39" V 2450 5800 50  0000 R CNN
 F 1 "Screw_Terminal_01x06" V 2350 6150 50  0000 R CNN
-F 2 "TerminalBlock_RND:TerminalBlock_RND_205-00005_1x06_P5.00mm_Horizontal" H 2250 5800 50  0001 C CNN
+F 2 "TerminalBlock_WAGO:TerminalBlock_WAGO_236-108_1x08_P5.00mm_45Degree" H 2250 5800 50  0001 C CNN
 F 3 "~" H 2250 5800 50  0001 C CNN
 	1    2250 5800
@@
 F 0 "J42" V 1400 6550 50  0000 R CNN
 F 1 "Screw_Terminal_01x06" V 1300 6900 50  0000 R CNN
-F 2 "TerminalBlock_RND:TerminalBlock_RND_205-00005_1x06_P5.00mm_Horizontal" H 1200 6550 50  0001 C CNN
+F 2 "TerminalBlock_WAGO:TerminalBlock_WAGO_236-108_1x08_P5.00mm_45Degree" H 1200 6550 50  0001 C CNN
 F 3 "~" H 1200 6550 50  0001 C CNN
 	1    1200 6550
@@
 F 0 "J43" V 2450 6550 50  0000 R CNN
 F 1 "Screw_Terminal_01x06" V 2350 6900 50  0000 R CNN
-F 2 "TerminalBlock_RND:TerminalBlock_RND_205-00005_1x06_P5.00mm_Horizontal" H 2250 6550 50  0001 C CNN
+F 2 "TerminalBlock_WAGO:TerminalBlock_WAGO_236-108_1x08_P5.00mm_45Degree" H 2250 6550 50  0001 C CNN
 F 3 "~" H 2250 6550 50  0001 C CNN
 	1    2250 6550
@@
 F 0 "J44" V 1967 7246 50  0000 C CNN
 F 1 "Screw_Terminal_01x12" V 1876 7246 50  0000 C CNN
-F 2 "TerminalBlock_RND:TerminalBlock_RND_205-00011_1x12_P5.00mm_Horizontal" H 1750 7300 50  0001 C CNN
+F 2 "TerminalBlock_WAGO:TerminalBlock_WAGO_236-112_1x12_P5.00mm_45Degree" H 1750 7300 50  0001 C CNN
 F 3 "~" H 1750 7300 50  0001 C CNN
 	1    1750 7300
@@
 F 0 "J22" V 11100 3350 50  0000 L CNN
 F 1 "12V Out" V 11200 3250 50  0000 L CNN
-F 2 "TerminalBlock_Altech:Altech_AK300_1x02_P5.00mm_45-Degree" H 11000 3450 50  0001 C CNN
+F 2 "TerminalBlock_WAGO:TerminalBlock_WAGO_236-102_1x02_P5.00mm_45Degree" H 11000 3450 50  0001 C CNN
 F 3 "https://datasheet.lcsc.com/lcsc/2106062140_DEGSON-DG129-5-08-02P-14-00A-H_C2760670.pdf" H 11000 3450 50  0001 C CNN
 	1    11000 3450
@@
 F 0 "J37" V 11100 5350 50  0000 L CNN
 F 1 "3.3V Out" V 11200 5250 50  0000 L CNN
-F 2 "TerminalBlock_Altech:Altech_AK300_1x02_P5.00mm_45-Degree" H 11000 5450 50  0001 C CNN
+F 2 "TerminalBlock_WAGO:TerminalBlock_WAGO_236-102_1x02_P5.00mm_45Degree" H 11000 5450 50  0001 C CNN
 F 3 "https://datasheet.lcsc.com/lcsc/2106062140_DEGSON-DG129-5-08-02P-14-00A-H_C2760670.pdf" H 11000 5450 50  0001 C CNN
 	1    11000 5450
@@
 F 0 "R7" H 8300 3000 50  0000 L CNN
 F 1 "680" V 8250 2950 50  0000 L CNN
-F 2 "Resistor_THT:R_Axial_Power_L20.0mm_W6.4mm_P25.40mm" V 8180 3000 50  0001 C CNN
+F 2 "Resistor_THT:R_Axial_DIN0516_L15.5mm_D5.0mm_P20.32mm_Horizontal" V 8180 3000 50  0001 C CNN
 F 3 "~" H 8250 3000 50  0001 C CNN
 	1    8250 3000
@@
 F 0 "J35" V 7150 5350 50  0000 L CNN
 F 1 "5V Out" V 7250 5250 50  0000 L CNN
-F 2 "TerminalBlock_Altech:Altech_AK300_1x02_P5.00mm_45-Degree" H 7050 5450 50  0001 C CNN
+F 2 "TerminalBlock_WAGO:TerminalBlock_WAGO_236-102_1x02_P5.00mm_45Degree" H 7050 5450 50  0001 C CNN
 F 3 "https://datasheet.lcsc.com/lcsc/2106062140_DEGSON-DG129-5-08-02P-14-00A-H_C2760670.pdf" H 7050 5450 50  0001 C CNN
 	1    7050 5450
@@
 F 0 "J20" V 7150 3350 50  0000 L CNN
 F 1 "12V Out" V 7250 3250 50  0000 L CNN
-F 2 "TerminalBlock_Altech:Altech_AK300_1x02_P5.00mm_45-Degree" H 7050 3450 50  0001 C CNN
+F 2 "TerminalBlock_WAGO:TerminalBlock_WAGO_236-102_1x02_P5.00mm_45Degree" H 7050 3450 50  0001 C CNN
 F 3 "https://datasheet.lcsc.com/lcsc/2106062140_DEGSON-DG129-5-08-02P-14-00A-H_C2760670.pdf" H 7050 3450 50  0001 C CNN
 	1    7050 3450
@@
 F 0 "J8" V 11100 1350 50  0000 L CNN
 F 1 "12V Out" V 11200 1250 50  0000 L CNN
-F 2 "TerminalBlock_Altech:Altech_AK300_1x02_P5.00mm_45-Degree" H 11000 1450 50  0001 C CNN
+F 2 "TerminalBlock_WAGO:TerminalBlock_WAGO_236-102_1x02_P5.00mm_45Degree" H 11000 1450 50  0001 C CNN
 F 3 "https://datasheet.lcsc.com/lcsc/2106062140_DEGSON-DG129-5-08-02P-14-00A-H_C2760670.pdf" H 11000 1450 50  0001 C CNN
 	1    11000 1450

Commit message: More pcb layout
Parts:
- J10: value EPS12V 8 Pin -> ATX12V1 8 Pin
- J13: value Molex: 0039281243 -> 12V2
- J4: value EPS12V 4Pin -> ATX12V1
Changed lines of the file:
@@
 AR Path="/5E13FF9B/62088F4B" Ref="J?"  Part="1"
 F 0 "J10" H 3000 1200 50  0000 C CNN
-F 1 "EPS12V 8 Pin" H 3000 1300 50  0000 C CNN
+F 1 "ATX12V1 8 Pin" H 3000 1300 50  0000 C CNN
 F 2 "Connector_Molex:Molex_Mini-Fit_Jr_5566-08A_2x04_P4.20mm_Vertical" H 2950 1600 50  0001 C CNN
 F 3 "https://www.molex.com/pdm_docs/sd/039281243_sd.pdf" H 2950 1600 50  0001 C CNN
@@
 P 2950 950
 F 0 "J4" H 3000 625 50  0000 C CNN
-F 1 "EPS12V 4Pin" H 3000 716 50  0000 C CNN
+F 1 "ATX12V1" H 3000 716 50  0000 C CNN
 F 2 "Connector_Molex:Molex_Mini-Fit_Jr_5566-04A_2x02_P4.20mm_Vertical" H 2950 950 50  0001 C CNN
 F 3 "~" H 2950 950 50  0001 C CNN
@@
 AR Path="/5E13FF9B/6241F25C" Ref="J?"  Part="1"
 F 0 "J13" H 2400 2850 50  0000 C CNN
-F 1 "Molex: 0039281243" V 2400 3300 39  0000 C CNN
+F 1 "12V2" V 2400 3300 39  0000 C CNN
 F 2 "Connector_Molex:Molex_Mini-Fit_Jr_5566-12A_2x06_P4.20mm_Vertical" H 2350 3350 50  0001 C CNN
 F 3 "https://www.molex.com/pdm_docs/sd/039281243_sd.pdf" H 2350 3350 50  0001 C CNN

Commit message: More pcb layout
Parts:
- R1, R10, R11, R12, R3, R5, R6, R7, R8, R9: footprint Resistor_THT:R_Axial_DIN0516_L15.5mm_D5.0mm_P20.32mm_Horizontal -> Resistor_SMD:R_2816_7142Metric_Pad3.20x4.45mm_HandSolder
Changed lines of the file:
@@
 F 0 "R8" H 9000 3000 50  0000 L CNN
 F 1 "1k" V 9150 2950 50  0000 L CNN
-F 2 "Resistor_THT:R_Axial_DIN0516_L15.5mm_D5.0mm_P20.32mm_Horizontal" V 9080 3000 50  0001 C CNN
+F 2 "Resistor_SMD:R_2816_7142Metric_Pad3.20x4.45mm_HandSolder" V 9080 3000 50  0001 C CNN
 F 3 "~" H 9150 3000 50  0001 C CNN
 	1    9150 3000
@@
 F 0 "R7" H 8300 3000 50  0000 L CNN
 F 1 "680" V 8250 2950 50  0000 L CNN
-F 2 "Resistor_THT:R_Axial_DIN0516_L15.5mm_D5.0mm_P20.32mm_Horizontal" V 8180 3000 50  0001 C CNN
+F 2 "Resistor_SMD:R_2816_7142Metric_Pad3.20x4.45mm_HandSolder" V 8180 3000 50  0001 C CNN
 F 3 "~" H 8250 3000 50  0001 C CNN
 	1    8250 3000
@@
 F 0 "R11" H 8000 5000 50  0000 L CNN
 F 1 "20" V 7950 4950 50  0000 L CNN
-F 2 "Resistor_THT:R_Axial_DIN0516_L15.5mm_D5.0mm_P20.32mm_Horizontal" V 7880 5000 50  0001 C CNN
+F 2 "Resistor_SMD:R_2816_7142Metric_Pad3.20x4.45mm_HandSolder" V 7880 5000 50  0001 C CNN
 F 3 "~" H 7950 5000 50  0001 C CNN
 	1    7950 5000
@@
 F 0 "R12" H 8650 5000 50  0000 L CNN
 F 1 "1k" V 8850 4950 50  0000 L CNN
-F 2 "Resistor_THT:R_Axial_DIN0516_L15.5mm_D5.0mm_P20.32mm_Horizontal" V 8780 5000 50  0001 C CNN
+F 2 "Resistor_SMD:R_2816_7142Metric_Pad3.20x4.45mm_HandSolder" V 8780 5000 50  0001 C CNN
 F 3 "~" H 8850 5000 50  0001 C CNN
 	1    8850 5000
@@
 F 0 "R9" H 4050 5000 50  0000 L CNN
 F 1 "300" V 4000 4950 50  0000 L CNN
-F 2 "Resistor_THT:R_Axial_DIN0516_L15.5mm_D5.0mm_P20.32mm_Horizontal" V 3930 5000 50  0001 C CNN
+F 2 "Resistor_SMD:R_2816_7142Metric_Pad3.20x4.45mm_HandSolder" V 3930 5000 50  0001 C CNN
 F 3 "~" H 4000 5000 50  0001 C CNN
 	1    4000 5000
@@
 F 0 "R10" H 4700 5000 50  0000 L CNN
 F 1 "1k" V 4900 4950 50  0000 L CNN
-F 2 "Resistor_THT:R_Axial_DIN0516_L15.5mm_D5.0mm_P20.32mm_Horizontal" V 4830 5000 50  0001 C CNN
+F 2 "Resistor_SMD:R_2816_7142Metric_Pad3.20x4.45mm_HandSolder" V 4830 5000 50  0001 C CNN
 F 3 "~" H 4900 5000 50  0001 C CNN
 	1    4900 5000
@@
 F 0 "R5" H 4350 3000 50  0000 L CNN
 F 1 "680" V 4300 2950 50  0000 L CNN
-F 2 "Resistor_THT:R_Axial_DIN0516_L15.5mm_D5.0mm_P20.32mm_Horizontal" V 4230 3000 50  0001 C CNN
+F 2 "Resistor_SMD:R_2816_7142Metric_Pad3.20x4.45mm_HandSolder" V 4230 3000 50  0001 C CNN
 F 3 "~" H 4300 3000 50  0001 C CNN
 	1    4300 3000
@@
 F 0 "R6" H 5050 3000 50  0000 L CNN
 F 1 "1k" V 5200 2950 50  0000 L CNN
-F 2 "Resistor_THT:R_Axial_DIN0516_L15.5mm_D5.0mm_P20.32mm_Horizontal" V 5130 3000 50  0001 C CNN
+F 2 "Resistor_SMD:R_2816_7142Metric_Pad3.20x4.45mm_HandSolder" V 5130 3000 50  0001 C CNN
 F 3 "~" H 5200 3000 50  0001 C CNN
 	1    5200 3000
@@
 F 0 "R1" H 7700 1000 50  0000 L CNN
 F 1 "680" V 7650 950 50  0000 L CNN
-F 2 "Resistor_THT:R_Axial_DIN0516_L15.5mm_D5.0mm_P20.32mm_Horizontal" V 7580 1000 50  0001 C CNN
+F 2 "Resistor_SMD:R_2816_7142Metric_Pad3.20x4.45mm_HandSolder" V 7580 1000 50  0001 C CNN
 F 3 "~" H 7650 1000 50  0001 C CNN
 	1    7650 1000
@@
 F 0 "R3" H 8700 1000 50  0000 L CNN
 F 1 "1k" V 8850 950 50  0000 L CNN
-F 2 "Resistor_THT:R_Axial_DIN0516_L15.5mm_D5.0mm_P20.32mm_Horizontal" V 8780 1000 50  0001 C CNN
+F 2 "Resistor_SMD:R_2816_7142Metric_Pad3.20x4.45mm_HandSolder" V 8780 1000 50  0001 C CNN
 F 3 "~" H 8850 1000 50  0001 C CNN
 	1    8850 1000

Commit message: densified circuit, defined edge cut, added mounting holes
Parts:
- R4: footprint Resistor_THT:R_Axial_DIN0516_L15.5mm_D5.0mm_P20.32mm_Horizontal -> Resistor_SMD:R_2816_7142Metric_Pad3.20x4.45mm_HandSolder
Changed lines of the file:
@@
 F 0 "R4" H 5650 1350 50  0000 L CNN
 F 1 "680" V 5600 1300 50  0000 L CNN
-F 2 "Resistor_THT:R_Axial_DIN0516_L15.5mm_D5.0mm_P20.32mm_Horizontal" V 5530 1350 50  0001 C CNN
+F 2 "Resistor_SMD:R_2816_7142Metric_Pad3.20x4.45mm_HandSolder" V 5530 1350 50  0001 C CNN
 F 3 "~" H 5600 1350 50  0001 C CNN
 	1    5600 1350

Commit message: cleanup
Parts:
- removed HS1: Heatsink, Heatsink:Heatsink_Stonecold_HS-132_32x14mm_2xFixation1.5mm, symbol Mechanical:Heatsink_Pad
- J38, J39, J42, J43: footprint TerminalBlock_WAGO:TerminalBlock_WAGO_236-108_1x08_P5.00mm_45Degree -> TerminalBlock_WAGO:TerminalBlock_WAGO_236-106_1x06_P5.00mm_45Degree
Other:
- note removed: "Mosfet Cooling"
- note removed: "The heatsink will be attached\nto the power mosfets."
Changed lines of the file:
@@
 F 0 "J38" V 1400 5800 50  0000 R CNN
 F 1 "Screw_Terminal_01x06" V 1300 6150 50  0000 R CNN
-F 2 "TerminalBlock_WAGO:TerminalBlock_WAGO_236-108_1x08_P5.00mm_45Degree" H 1200 5800 50  0001 C CNN
+F 2 "TerminalBlock_WAGO:TerminalBlock_WAGO_236-106_1x06_P5.00mm_45Degree" H 1200 5800 50  0001 C CNN
 F 3 "~" H 1200 5800 50  0001 C CNN
 	1    1200 5800
@@
 F 0 "J39" V 2450 5800 50  0000 R CNN
 F 1 "Screw_Terminal_01x06" V 2350 6150 50  0000 R CNN
-F 2 "TerminalBlock_WAGO:TerminalBlock_WAGO_236-108_1x08_P5.00mm_45Degree" H 2250 5800 50  0001 C CNN
+F 2 "TerminalBlock_WAGO:TerminalBlock_WAGO_236-106_1x06_P5.00mm_45Degree" H 2250 5800 50  0001 C CNN
 F 3 "~" H 2250 5800 50  0001 C CNN
 	1    2250 5800
@@
 F 0 "J42" V 1400 6550 50  0000 R CNN
 F 1 "Screw_Terminal_01x06" V 1300 6900 50  0000 R CNN
-F 2 "TerminalBlock_WAGO:TerminalBlock_WAGO_236-108_1x08_P5.00mm_45Degree" H 1200 6550 50  0001 C CNN
+F 2 "TerminalBlock_WAGO:TerminalBlock_WAGO_236-106_1x06_P5.00mm_45Degree" H 1200 6550 50  0001 C CNN
 F 3 "~" H 1200 6550 50  0001 C CNN
 	1    1200 6550
@@
 F 0 "J43" V 2450 6550 50  0000 R CNN
 F 1 "Screw_Terminal_01x06" V 2350 6900 50  0000 R CNN
-F 2 "TerminalBlock_WAGO:TerminalBlock_WAGO_236-108_1x08_P5.00mm_45Degree" H 2250 6550 50  0001 C CNN
+F 2 "TerminalBlock_WAGO:TerminalBlock_WAGO_236-106_1x06_P5.00mm_45Degree" H 2250 6550 50  0001 C CNN
 F 3 "~" H 2250 6550 50  0001 C CNN
 	1    2250 6550
@@
 	0    -1   1    0
 $EndComp
-$Comp
-L Graphic:SYM_Hot_Small #SYM1
-U 1 1 62592F2B
-P 6600 950
-F 0 "#SYM1" H 6600 1090 50  0001 C CNN
-F 1 "SYM_Hot_Small" H 6600 825 50  0001 C CNN
-F 2 "" H 6600 775 50  0001 C CNN
-F 3 "~" H 6630 750 50  0001 C CNN
-	1    6600 950
-	1    0    0    -1
-$EndComp
-$Comp
-L Mechanical:Heatsink_Pad HS1
-U 1 1 62592F31
-P 6600 1150
-F 0 "HS1" H 6250 1250 50  0000 L CNN
-F 1 "Heatsink" H 6150 1150 50  0000 L CNN
-F 2 "Heatsink:Heatsink_Stonecold_HS-132_32x14mm_2xFixation1.5mm" H 6612 1100 50  0001 C CNN
-F 3 "~" H 6612 1100 50  0001 C CNN
-	1    6600 1150
-	1    0    0    -1
-$EndComp
 Wire Wire Line
 	10050 5650 10050 5750
@@
 Wire Wire Line
 	8250 3550 8500 3550
-$Comp
-L power:GNDREF #PWR06
-U 1 1 627177F1
-P 6600 1250
-F 0 "#PWR06" H 6600 1000 50  0001 C CNN
-F 1 "GNDREF" H 6605 1077 50  0000 C CNN
-F 2 "" H 6600 1250 50  0001 C CNN
-F 3 "" H 6600 1250 50  0001 C CNN
-	1    6600 1250
-	1    0    0    -1
-$EndComp
 $Comp
 L Connector_Generic:Conn_01x02 J29
@@
 Wire Notes Line
 	6050 550  4950 550
-Wire Notes Line
-	6100 550  6100 2200
-Wire Notes Line
-	6100 2200 6900 2200
-Wire Notes Line
-	6900 2200 6900 550
-Wire Notes Line
-	6900 550  6100 550
 Text Notes 3850 2150 0    30   ~ 0
 Connect a swst switch.\nThe switch will short the PS_ON connector \nwith the Ground and start the power supply.\n\nWhen using a switch with LED lighting then\nuse a one of the power rails to power the\nled seperately and put a pull-up resistor\ninto your led circuit.
@@
 Text Notes 5150 650  0    50   ~ 0
 Standby Indicator
-Text Notes 6150 1850 0    30   ~ 0
-The heatsink will be attached\nto the power mosfets.
-Text Notes 6200 650  0    50   ~ 0
-Mosfet Cooling
 Wire Wire Line
 	2100 4900 2100 4800

Commit message: refit traces, added global label added text
Connections:
- net +F5V: now reaches DZ4.1 (K), F4.2, J28.1 (Pin_1), R10.2, R9.1, U4.1 (IP+), U4.2 (IP+)
Changed lines of the file:
@@
 	9550 3250 9550 3650
 Text GLabel 9500 3250 0    50   Input ~ 0
-+5V
++5VF
 Wire Wire Line
 	9950 3650 9950 3950
@@
 	9550 5250 9550 5650
 Text GLabel 9500 5250 0    50   Input ~ 0
-+5V
++5VF
 Wire Wire Line
 	9950 5650 9950 5950
@@
 	1    0    0    -1
 $EndComp
-$Comp
-L power:GNDREF #PWR028
-U 1 1 62592F9F
-P 5150 5050
-F 0 "#PWR028" H 5150 4800 50  0001 C CNN
-F 1 "GNDREF" H 5155 4877 50  0000 C CNN
-F 2 "" H 5150 5050 50  0001 C CNN
-F 3 "" H 5150 5050 50  0001 C CNN
-	1    5150 5050
-	1    0    0    -1
-$EndComp
 Wire Wire Line
 	4700 5550 4700 5450
@@
 	6000 5650 6000 5950
 Text GLabel 5550 5250 0    50   Input ~ 0
-+5V
++5VF
 Wire Wire Line
 	5600 5250 5600 5650
@@
 	6000 3650 6000 3950
 Text GLabel 5550 3250 0    50   Input ~ 0
-+5V
++5VF
 Wire Wire Line
 	5600 3250 5600 3650
@@
 	9950 1650 9950 1950
 Text GLabel 9500 1250 0    50   Input ~ 0
-+5V
++5VF
 Wire Wire Line
 	9550 1250 9550 1650
@@
 	0    -1   -1   0
 $EndComp
+Text GLabel 4000 4850 1    50   Output ~ 0
++F5V
+$Comp
+L power:GNDREF #PWR028
+U 1 1 62592F9F
+P 5150 5050
+F 0 "#PWR028" H 5150 4800 50  0001 C CNN
+F 1 "GNDREF" H 5155 4877 50  0000 C CNN
+F 2 "" H 5150 5050 50  0001 C CNN
+F 3 "" H 5150 5050 50  0001 C CNN
+	1    5150 5050
+	1    0    0    -1
+$EndComp
 $EndSCHEMATC
