File: KiCAD/ATX_PSU_525W_ENERMAX/ATX_PSDB.sch (KiCad schematic (older format))
At the start: 86 parts, among them J1 Fan1, J10 ATX12V1 8 Pin, J11 Current Sens, J12 Molex: 0039281243, J13 12V2, J14 Molex: 0039281243, J15 Potti, J16 Potti, J17 LED Yellow, J18 LED Yellow, J19 Volt Sens, J2 Power On Switch, J20 12V Out, J21 Volt Sens, J22 12V Out, J23 Molex: 0039281243, J24 Current Sens, J25 Current Sens, J26 Molex: 0039281243, J27 Molex: 0039281243, J28 Fan1, J29 Fan1, J3 Standby LED, J30 Potti, J31 Potti, J32 LED Red, J33 LED Orange, J34 Volt Sens, J35 5V Out, J36 Volt Sens, J37 3.3V Out, J38 Screw_Terminal_01x06, J39 Screw_Terminal_01x06, J4 ATX12V1, J40 Current Sens, J41 Current Sens, J42 Screw_Terminal_01x06, J43 Screw_Terminal_01x06, J44 Screw_Terminal_01x12, J5 Potti, J6 LED Yellow, J7 Volt Sens, J8 12V Out, J9 Main ATX 24Pin, Q1 Q_NMOS_DGS, Q2 Q_NMOS_DGS, Q3 Q_NMOS_DGS, Q4 Q_NMOS_DGS, Q5 Q_NMOS_DGS, U1 ACS712xLCTR-20A, U2 ACS712xLCTR-20A, U3 ACS712xLCTR-20A, U4 ACS712xLCTR-20A, U5 ACS712xLCTR-20A

Commit message: Corrections and so on
Parts:
- J10: value ATX12V1 8 Pin -> ATX 12V1 Input
- J12, J14: value Molex: 0039281243 -> Molex: ATX 12V2 Input
- J13: value 12V2 -> Molex: ATX 12V2 Input
- J23, J26, J27: value Molex: 0039281243 -> Molex: ATX 12V3 Input
- J38: value Screw_Terminal_01x06 -> Terminal: +12V2 Input
- J39: value Screw_Terminal_01x06 -> Terminal: +12V3 Input
- J4: value ATX12V1 -> ATX 12V1 Input
- J42: value Screw_Terminal_01x06 -> Terminal: +5V Input
- J43: value Screw_Terminal_01x06 -> Terminal: +3.3V Input
- J44: value Screw_Terminal_01x12 -> Terminal: Ground
Connections:
- net +F5V is gone; now on net +5V: DZ4.1 (K), F4.2, J28.1 (Pin_1), R10.2, R9.1, U4.1 (IP+), U4.2 (IP+)
Changed lines of the file:
@@
 AR Path="/5E13FF9B/62088F4B" Ref="J?"  Part="1"
 F 0 "J10" H 3000 1200 50  0000 C CNN
-F 1 "ATX12V1 8 Pin" H 3000 1300 50  0000 C CNN
+F 1 "ATX 12V1 Input" H 3000 1300 50  0001 C CNN
 F 2 "Connector_Molex:Molex_Mini-Fit_Jr_5566-08A_2x04_P4.20mm_Vertical" H 2950 1600 50  0001 C CNN
 F 3 "https://www.molex.com/pdm_docs/sd/039281243_sd.pdf" H 2950 1600 50  0001 C CNN
@@
 P 1200 5800
 F 0 "J38" V 1400 5800 50  0000 R CNN
-F 1 "Screw_Terminal_01x06" V 1300 6150 50  0000 R CNN
+F 1 "Terminal: +12V2 Input" V 1300 6150 50  0000 R CNN
 F 2 "TerminalBlock_WAGO:TerminalBlock_WAGO_236-106_1x06_P5.00mm_45Degree" H 1200 5800 50  0001 C CNN
 F 3 "~" H 1200 5800 50  0001 C CNN
@@
 P 2250 5800
 F 0 "J39" V 2450 5800 50  0000 R CNN
-F 1 "Screw_Terminal_01x06" V 2350 6150 50  0000 R CNN
+F 1 "Terminal: +12V3 Input" V 2350 6150 50  0000 R CNN
 F 2 "TerminalBlock_WAGO:TerminalBlock_WAGO_236-106_1x06_P5.00mm_45Degree" H 2250 5800 50  0001 C CNN
 F 3 "~" H 2250 5800 50  0001 C CNN
@@
 P 1200 6550
 F 0 "J42" V 1400 6550 50  0000 R CNN
-F 1 "Screw_Terminal_01x06" V 1300 6900 50  0000 R CNN
+F 1 "Terminal: +5V Input" V 1300 6900 50  0000 R CNN
 F 2 "TerminalBlock_WAGO:TerminalBlock_WAGO_236-106_1x06_P5.00mm_45Degree" H 1200 6550 50  0001 C CNN
 F 3 "~" H 1200 6550 50  0001 C CNN
@@
 P 2250 6550
 F 0 "J43" V 2450 6550 50  0000 R CNN
-F 1 "Screw_Terminal_01x06" V 2350 6900 50  0000 R CNN
+F 1 "Terminal: +3.3V Input" V 2350 6900 50  0000 R CNN
 F 2 "TerminalBlock_WAGO:TerminalBlock_WAGO_236-106_1x06_P5.00mm_45Degree" H 2250 6550 50  0001 C CNN
 F 3 "~" H 2250 6550 50  0001 C CNN
@@
 P 1750 7300
 F 0 "J44" V 1967 7246 50  0000 C CNN
-F 1 "Screw_Terminal_01x12" V 1876 7246 50  0000 C CNN
+F 1 "Terminal: Ground" V 1876 7246 50  0000 C CNN
 F 2 "TerminalBlock_WAGO:TerminalBlock_WAGO_236-112_1x12_P5.00mm_45Degree" H 1750 7300 50  0001 C CNN
 F 3 "~" H 1750 7300 50  0001 C CNN
@@
 U 1 1 620C0620
 P 2950 950
-F 0 "J4" H 3000 625 50  0000 C CNN
-F 1 "ATX12V1" H 3000 716 50  0000 C CNN
+F 0 "J4" H 3000 750 50  0000 C CNN
+F 1 "ATX 12V1 Input" H 3000 716 50  0001 C CNN
 F 2 "Connector_Molex:Molex_Mini-Fit_Jr_5566-04A_2x02_P4.20mm_Vertical" H 2950 950 50  0001 C CNN
 F 3 "~" H 2950 950 50  0001 C CNN
@@
 AR Path="/623260A0" Ref="J26"  Part="1"
 AR Path="/5E13FF9B/623260A0" Ref="J?"  Part="1"
-F 0 "J26" H 2350 4200 50  0000 C CNN
-F 1 "Molex: 0039281243" V 2350 4650 39  0000 C CNN
+F 0 "J26" H 2350 4300 50  0000 C CNN
+F 1 "Molex: ATX 12V3 Input" V 2350 4650 39  0001 C CNN
 F 2 "Connector_Molex:Molex_Mini-Fit_Jr_5566-12A_2x06_P4.20mm_Vertical" H 2300 4700 50  0001 C CNN
 F 3 "https://www.molex.com/pdm_docs/sd/039281243_sd.pdf" H 2300 4700 50  0001 C CNN
-F 4 "WM3811-ND " H 2400 4300 50  0000 C CNN "Digi-Key"
+F 4 "WM3811-ND " H 2400 4300 50  0001 C CNN "Digi-Key"
 	1    2300 4700
 	1    0    0    1
@@
 AR Path="/5E13FF9B/621ECDC3" Ref="J?"  Part="1"
 F 0 "J23" H 1200 4200 50  0000 C CNN
-F 1 "Molex: 0039281243" V 1200 4350 39  0001 C CNN
+F 1 "Molex: ATX 12V3 Input" V 1200 4350 39  0001 C CNN
 F 2 "Connector_Molex:Molex_Mini-Fit_Jr_5566-06A_2x03_P4.20mm_Vertical" H 1150 4400 50  0001 C CNN
 F 3 "https://www.molex.com/pdm_docs/sd/039281243_sd.pdf" H 1150 4400 50  0001 C CNN
@@
 AR Path="/5E13FF9B/621ECDE7" Ref="J?"  Part="1"
 F 0 "J27" H 1200 4750 50  0000 C CNN
-F 1 "Molex: 0039281243" V 1200 4900 39  0001 C CNN
+F 1 "Molex: ATX 12V3 Input" V 1200 4900 39  0001 C CNN
 F 2 "Connector_Molex:Molex_Mini-Fit_Jr_5566-06A_2x03_P4.20mm_Vertical" H 1150 4950 50  0001 C CNN
 F 3 "https://www.molex.com/pdm_docs/sd/039281243_sd.pdf" H 1150 4950 50  0001 C CNN
@@
 	9550 3250 9550 3650
 Text GLabel 9500 3250 0    50   Input ~ 0
-+5VF
++F5V
 Wire Wire Line
 	9950 3650 9950 3950
@@
 	9550 5250 9550 5650
 Text GLabel 9500 5250 0    50   Input ~ 0
-+5VF
++F5V
 Wire Wire Line
 	9950 5650 9950 5950
@@
 	6000 5650 6000 5950
 Text GLabel 5550 5250 0    50   Input ~ 0
-+5VF
++F5V
 Wire Wire Line
 	5600 5250 5600 5650
@@
 	6000 3650 6000 3950
 Text GLabel 5550 3250 0    50   Input ~ 0
-+5VF
++F5V
 Wire Wire Line
 	5600 3250 5600 3650
@@
 	9950 1650 9950 1950
 Text GLabel 9500 1250 0    50   Input ~ 0
-+5VF
++F5V
 Wire Wire Line
 	9550 1250 9550 1650
@@
 AR Path="/5E13FF9B/62196D36" Ref="J?"  Part="1"
 F 0 "J14" H 1200 3400 50  0000 C CNN
-F 1 "Molex: 0039281243" V 1200 3550 39  0001 C CNN
+F 1 "Molex: ATX 12V2 Input" V 1200 3550 39  0001 C CNN
 F 2 "Connector_Molex:Molex_Mini-Fit_Jr_5566-06A_2x03_P4.20mm_Vertical" H 1150 3600 50  0001 C CNN
 F 3 "https://www.molex.com/pdm_docs/sd/039281243_sd.pdf" H 1150 3600 50  0001 C CNN
@@
 AR Path="/6241F25C" Ref="J13"  Part="1"
 AR Path="/5E13FF9B/6241F25C" Ref="J?"  Part="1"
-F 0 "J13" H 2400 2850 50  0000 C CNN
-F 1 "12V2" V 2400 3300 39  0000 C CNN
+F 0 "J13" H 2400 2950 50  0000 C CNN
+F 1 "Molex: ATX 12V2 Input" V 2400 3300 39  0001 C CNN
 F 2 "Connector_Molex:Molex_Mini-Fit_Jr_5566-12A_2x06_P4.20mm_Vertical" H 2350 3350 50  0001 C CNN
 F 3 "https://www.molex.com/pdm_docs/sd/039281243_sd.pdf" H 2350 3350 50  0001 C CNN
-F 4 "WM3811-ND " H 2450 2950 50  0000 C CNN "Digi-Key"
+F 4 "WM3811-ND " H 2450 2950 50  0001 C CNN "Digi-Key"
 	1    2350 3350
 	1    0    0    1
@@
 AR Path="/5E13FF9B/61DC7D9B" Ref="J?"  Part="1"
 F 0 "J12" H 1200 2850 50  0000 C CNN
-F 1 "Molex: 0039281243" V 1200 3000 39  0001 C CNN
+F 1 "Molex: ATX 12V2 Input" V 1200 3000 39  0001 C CNN
 F 2 "Connector_Molex:Molex_Mini-Fit_Jr_5566-06A_2x03_P4.20mm_Vertical" H 1150 3050 50  0001 C CNN
 F 3 "https://www.molex.com/pdm_docs/sd/039281243_sd.pdf" H 1150 3050 50  0001 C CNN
