File: pcb/ATX_PSDB.kicad_pcb (KiCad board)
At the start: 2 copper layers, 160 x 170 mm, 91 parts, among them J1 Fan1, J10 ATX 12V1 Input, J11 Current Sens, J12 Molex: ATX 12V2 Input, J13 Molex: ATX 12V2 Input, J14 Molex: ATX 12V2 Input, J15 Potti, J16 Potti, J17 LED Yellow, J18 LED Yellow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

Commit message: cleanup
Parts:
- removed the G*** at (26.6, 33.3)
- added G***: ÍboschTonosch, CustomFootPrints:logo_iboschtonosch, F.Cu at (24.8, 35.1)

Commit message: Migrate to KiCad 6.0
Other:
- net class Default removed
